File: Controle_Motor_DC/Controle_Motor_DC/Controle_Motor_DC.kicad_sch (KiCad schematic)
At the start: 13 parts, among them K1 Relay_SPST-NO, M1 Motor_DC, Q1 BC140, SW1 SW_Push, SW2 SW_Push, U2 RC1602A, Y1 12MHz

Commit message: Adição dos arquivos gerber, atualização do README, adição da imagem do modelo 3D da placa
Parts:
- added BT1: 5V, Connector_BarrelJack:BarrelJack_CUI_PJ-063AH_Horizontal, symbol Device:Battery
- C1, C2: footprint (none) -> Capacitor_THT:C_Rect_L4.0mm_W2.5mm_P2.50mm
- C3: footprint (none) -> Capacitor_THT:CP_Radial_D5.0mm_P2.50mm
- K1: footprint (none) -> Controle_Motor_DC:Relay_COMUS_3570_1331
- M1: footprint (none) -> Connector_Phoenix_GMSTB:PhoenixContact_GMSTBV_2,5_2-GF-7,62_1x02_P7.62mm_Vertical_ThreadedFlange_MountHole
- R1: footprint (none) -> Resistor_THT:R_Axial_DIN0207_L6.3mm_D2.5mm_P7.62mm_Horizontal
- RV1: footprint (none) -> Potentiometer_THT:Potentiometer_ACP_CA6-H2,5_Horizontal
- SW1, SW2: footprint (none) -> Button_Switch_THT:SW_PUSH-12mm_Wuerth-430476085716
- U1: footprint (none) -> Controle_Motor_DC:AT89C51-PDIP
- Y1: footprint (none) -> Crystal:Resonator-2Pin_W10.0mm_H5.0mm
Connections:
- net GND: now also BT1.2 (-)
- net VCC: now also BT1.1 (+)
Changed lines of the file:
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@@
+    (stroke (width 0) (type default))
+  )
+  (wire (pts (xy 55.88 76.2) (xy 55.88 78.74))
     (stroke (width 0) (type default))
   )
@@
   )
   (wire (pts (xy 156.21 88.9) (xy 172.72 88.9))
+    (stroke (width 0) (type default))
+  )
+  (wire (pts (xy 55.88 88.9) (xy 55.88 92.71))
     (stroke (width 0) (type default))
   )
@@
     )
   )
+  (symbol (lib_id "Device:Battery") (at 55.88 83.82 0) (unit 1)
+    (in_bom yes) (on_board yes) (dnp no) (fields_autoplaced)
+    (property "Reference" "BT1" (at 59.69 81.9785 0)
+      (effects (font (size 1.27 1.27)) (justify left))
+    )
+    (property "Value" "5V" (at 59.69 84.5185 0)
+      (effects (font (size 1.27 1.27)) (justify left))
+    )
+    (property "Footprint" "Connector_BarrelJack:BarrelJack_CUI_PJ-063AH_Horizontal" (at 55.88 82.296 90)
+      (effects (font (size 1.27 1.27)) hide)
+    )
+    (property "Datasheet" "~" (at 55.88 82.296 90)
+      (effects (font (size 1.27 1.27)) hide)
+    )
+    (pin "1")
+    (pin "2")
+    (instances
+      (project "Controle_Motor_DC"
+        (path "/3c0be8a9-5618-4f6c-9785-37958cca7ae6"
+          (reference "BT1") (unit 1)
+        )
+      )
+    )
+  )
   (symbol (lib_id "Switch:SW_Push") (at 156.21 151.13 0) (mirror y) (unit 1)
     (in_bom yes) (on_board yes) (dnp no) (fields_autoplaced)
@@
       (effects (font (size 1.27 1.27)))
     )
-    (property "Footprint" "" (at 156.21 146.05 0)
+    (property "Footprint" "Button_Switch_THT:SW_PUSH-12mm_Wuerth-430476085716" (at 156.21 146.05 0)
       (effects (font (size 1.27 1.27)) hide)
     )
@@
       (effects (font (size 1.27 1.27)))
     )
-    (property "Footprint" "" (at 130.81 95.25 0)
+    (property "Footprint" "Controle_Motor_DC:AT89C51-PDIP" (at 130.81 95.25 0)
       (effects (font (size 1.27 1.27)) hide)
     )
@@
       (effects (font (size 1.27 1.27)) (justify right))
     )
-    (property "Footprint" "" (at 219.71 88.9 0)
+    (property "Footprint" "Potentiometer_THT:Potentiometer_ACP_CA6-H2,5_Horizontal" (at 219.71 88.9 0)
       (effects (font (size 1.27 1.27)) hide)
     )
@@
       (effects (font (size 1.27 1.27)) (justify right))
     )
-    (property "Footprint" "" (at 91.44 121.92 0)
+    (property "Footprint" "Crystal:Resonator-2Pin_W10.0mm_H5.0mm" (at 91.44 121.92 0)
       (effects (font (size 1.27 1.27)) hide)
     )
@@
       (effects (font (size 1.27 1.27)))
     )
-    (property "Footprint" "" (at 76.2 115.2652 0)
+    (property "Footprint" "Capacitor_THT:C_Rect_L4.0mm_W2.5mm_P2.50mm" (at 76.2 115.2652 0)
       (effects (font (size 1.27 1.27)) hide)
     )
@@
       (effects (font (size 1.27 1.27)) (justify right))
     )
-    (property "Footprint" "" (at 148.59 38.1 0)
+    (property "Footprint" "Button_Switch_THT:SW_PUSH-12mm_Wuerth-430476085716" (at 148.59 38.1 0)
       (effects (font (size 1.27 1.27)) hide)
     )
@@
         (path "/3c0be8a9-5618-4f6c-9785-37958cca7ae6"
           (reference "SW1") (unit 1)
+        )
+      )
+    )
+  )
+  (symbol (lib_id "power:GND") (at 55.88 92.71 0) (mirror y) (unit 1)
+    (in_bom yes) (on_board yes) (dnp no) (fields_autoplaced)
+    (property "Reference" "#PWR015" (at 55.88 99.06 0)
+      (effects (font (size 1.27 1.27)) hide)
+    )
+    (property "Value" "GND" (at 55.88 97.79 0)
+      (effects (font (size 1.27 1.27)))
+    )
+    (property "Footprint" "" (at 55.88 92.71 0)
+      (effects (font (size 1.27 1.27)) hide)
+    )
+    (property "Datasheet" "" (at 55.88 92.71 0)
+      (effects (font (size 1.27 1.27)) hide)
+    )
+    (pin "1")
+    (instances
+      (project "Controle_Motor_DC"
+        (path "/3c0be8a9-5618-4f6c-9785-37958cca7ae6"
+          (reference "#PWR015") (unit 1)
         )
       )
@@
       (effects (font (size 1.27 1.27)) (justify left))
     )
-    (property "Footprint" "" (at 130.048 50.8 90)
+    (property "Footprint" "Resistor_THT:R_Axial_DIN0207_L6.3mm_D2.5mm_P7.62mm_Horizontal" (at 130.048 50.8 90)
       (effects (font (size 1.27 1.27)) hide)
     )
@@
       (effects (font (size 1.27 1.27)))
     )
-    (property "Footprint" "" (at 115.57 185.42 0)
+    (property "Footprint" "Controle_Motor_DC:Relay_COMUS_3570_1331" (at 115.57 185.42 0)
       (effects (font (size 1.27 1.27)) (justify left) hide)
     )
@@
       (effects (font (size 1.27 1.27)))
     )
-    (property "Footprint" "" (at 143.256 181.61 0)
+    (property "Footprint" "Connector_Phoenix_GMSTB:PhoenixContact_GMSTBV_2,5_2-GF-7,62_1x02_P7.62mm_Vertical_ThreadedFlange_MountHole" (at 143.256 181.61 0)
       (effects (font (size 1.27 1.27)) hide)
     )
@@
       (effects (font (size 1.27 1.27)))
     )
-    (property "Footprint" "" (at 76.2 130.5052 0)
+    (property "Footprint" "Capacitor_THT:C_Rect_L4.0mm_W2.5mm_P2.50mm" (at 76.2 130.5052 0)
       (effects (font (size 1.27 1.27)) hide)
     )
@@
       (effects (font (size 1.27 1.27)) (justify left))
     )
-    (property "Footprint" "" (at 127.3048 43.18 0)
+    (property "Footprint" "Capacitor_THT:CP_Radial_D5.0mm_P2.50mm" (at 127.3048 43.18 0)
       (effects (font (size 1.27 1.27)) hide)
     )
@@
         )
       )
+    )
+  )
+  (symbol (lib_id "power:VCC") (at 55.88 76.2 0) (unit 1)
+    (in_bom yes) (on_board yes) (dnp no) (fields_autoplaced)
+    (property "Reference" "#PWR016" (at 55.88 80.01 0)
+      (effects (font (size 1.27 1.27)) hide)
+    )
+    (property "Value" "VCC" (at 55.88 71.12 0)
+      (effects (font (size 1.27 1.27)))
+    )
+    (property "Footprint" "" (at 55.88 76.2 0)
+      (effects (font (size 1.27 1.27)) hide)
+    )
+    (property "Datasheet" "" (at 55.88 76.2 0)
+      (effects (font (size 1.27 1.27)) hide)
+    )
+    (pin "1")
+    (instances
+      (project "Controle_Motor_DC"
+        (path "/3c0be8a9-5618-4f6c-9785-37958cca7ae6"
+          (reference "#PWR016") (unit 1)
+        )
+      )
